Commit message: joint type changed to revolute

File: sef_roboter_support/urdf/sr25_macro.xacro (robot description, xacro)
@@ -166,5 +166,5 @@
 			<child link="base_link"/>
 	      </joint>
-	      <joint name="${prefix}joint_1" type="continuous">
+	      <joint name="${prefix}joint_1" type="revolute">
 			<parent link="${prefix}base_link"/>
 			<child link="${prefix}link_1"/>
@@ -174,5 +174,5 @@
  			<dynamics damping="0.7" friction="100"/>
 	      </joint>
-	      <joint name="${prefix}joint_2" type="continuous">
+	      <joint name="${prefix}joint_2" type="revolute">
 			<parent link="${prefix}link_1"/>
 			<child link="${prefix}link_2"/>
@@ -182,5 +182,5 @@
 			<dynamics damping="0.7" friction="100"/>
 	      </joint>
-	      <joint name="${prefix}joint_3" type="continuous">
+	      <joint name="${prefix}joint_3" type="revolute">
 			<parent link="${prefix}link_2"/>
 			<child link="${prefix}link_3"/>
@@ -190,5 +190,5 @@
 		        <dynamics damping="0.7" friction="100"/>
 	      </joint>
-	      <joint name="${prefix}joint_4" type="continuous">
+	      <joint name="${prefix}joint_4" type="revolute">
 			<parent link="${prefix}link_3"/>
 			<child link="${prefix}link_4"/>
@@ -198,5 +198,5 @@
 			<dynamics damping="0.7" friction="100"/>
               </joint>
-	      <joint name="${prefix}joint_5" type="continuous">
+	      <joint name="${prefix}joint_5" type="revolute">
 			<parent link="${prefix}link_4"/>
 			<child link="${prefix}link_5"/>
@@ -206,5 +206,5 @@
 			<dynamics damping="0.7" friction="100"/>
               </joint>
-	      <joint name="${prefix}joint_6" type="continuous">
+	      <joint name="${prefix}joint_6" type="revolute">
 			<parent link="${prefix}link_5"/>
 			<child link="${prefix}link_tool"/>

Commit message: adopting for full 6 axis ros_control

File: sef_roboter_support/urdf/sr25_macro.xacro (robot description, xacro)
@@ -171,5 +171,5 @@
 			<origin xyz="0 0 0.075738" rpy="1.5708 0 -1.5745"/>
 			<axis xyz="0 -1 0" />
-			<limit lower="-2.8" upper="2.8" effort="10000" velocity="2" />
+			<limit lower="-2.8" upper="2.8" effort="10000" velocity="1" />
  			<dynamics damping="0.7" friction="100"/>
 	      </joint>
@@ -179,5 +179,5 @@
 			<origin xyz="0 0.24264 -0.29599" rpy="1.5687 0 0"/>
 			<axis xyz="-1 0 0" />
-			<limit lower="-0.5" upper="1.5" effort="10000" velocity="2" />
+			<limit lower="-0.5" upper="1.5" effort="10000" velocity="1" />
 			<dynamics damping="0.7" friction="100"/>
 	      </joint>
@@ -187,5 +187,5 @@
 			<origin xyz="0 0 -0.79724" rpy="0.005529 0 0"/>
 			<axis xyz="-1 0 0" />
-			<limit lower="-0.5" upper="1.5" effort="10000" velocity="2" />
+			<limit lower="-0.5" upper="1.5" effort="10000" velocity="1" />
 		        <dynamics damping="0.7" friction="100"/>
 	      </joint>
@@ -195,5 +195,5 @@
 			<origin xyz="0 -0.15811 0" rpy="0 0.0014787 0"/>
 			<axis xyz="0 1 0" />
-			<limit lower="-1.6" upper="1.6" effort="10000" velocity="2" />
+			<limit lower="-1.6" upper="1.6" effort="10000" velocity="1" />
 			<dynamics damping="0.7" friction="100"/>
               </joint>
@@ -203,5 +203,5 @@
 			<origin xyz="0 -0.58433 0" rpy="0 0 -0.033693"/>
 			<axis xyz="0 0 1" />
-			<limit lower="-3" upper="3" effort="10000" velocity="2" />
+			<limit lower="-3" upper="3" effort="10000" velocity="1" />
 			<dynamics damping="0.7" friction="100"/>
               </joint>

Commit message: fixing joint limits

File: sef_roboter_support/urdf/sr25_macro.xacro (robot description, xacro)
@@ -179,5 +179,5 @@
 			<origin xyz="0 0.24264 -0.29599" rpy="1.5687 0 0"/>
 			<axis xyz="-1 0 0" />
-			<limit lower="-0.5" upper="1.5" effort="10000" velocity="1" />
+                        <limit lower="-0.5" upper="1.5" effort="10000" velocity="1" />
 			<dynamics damping="0.7" friction="100"/>
 	      </joint>
@@ -187,5 +187,5 @@
 			<origin xyz="0 0 -0.79724" rpy="0.005529 0 0"/>
 			<axis xyz="-1 0 0" />
-			<limit lower="-0.5" upper="1.5" effort="10000" velocity="1" />
+                        <limit lower="-1.5" upper="0.5" effort="10000" velocity="1" />
 		        <dynamics damping="0.7" friction="100"/>
 	      </joint>
@@ -195,5 +195,5 @@
 			<origin xyz="0 -0.15811 0" rpy="0 0.0014787 0"/>
 			<axis xyz="0 1 0" />
-			<limit lower="-1.6" upper="1.6" effort="10000" velocity="1" />
+                        <limit lower="-3" upper="3" effort="10000" velocity="1" />
 			<dynamics damping="0.7" friction="100"/>
               </joint>
@@ -203,5 +203,5 @@
 			<origin xyz="0 -0.58433 0" rpy="0 0 -0.033693"/>
 			<axis xyz="0 0 1" />
-			<limit lower="-3" upper="3" effort="10000" velocity="1" />
+                        <limit lower="-1.6" upper="1.6" effort="10000" velocity="1" />
 			<dynamics damping="0.7" friction="100"/>
               </joint>

Commit message: changing black color of joints to grey

File: sef_roboter_support/urdf/sr25_macro.xacro (robot description, xacro)
@@ -10,5 +10,5 @@
 				    <mesh filename="package://sef_roboter_support/meshes/sr25/visual/sr25_base_axis.stl" />
 			      </geometry>
-			      <material name="black"/>
+            <material name="grey"/>
 		      </visual>
 		      <collision>
@@ -33,5 +33,5 @@
 				    <mesh filename="package://sef_roboter_support/meshes/sr25/visual/sr25_axis_1.stl"  />
 			      </geometry>
-			      <material name="black"/>
+            <material name="grey"/>
 		      </visual>
 		      <collision>
@@ -77,5 +77,5 @@
 				    <mesh filename="package://sef_roboter_support/meshes/sr25/visual/sr25_axis_3.stl" />
 			      </geometry>
-			      <material name="black" />
+            <material name="grey" />
 		      </visual>
 		      <collision>
@@ -143,5 +143,5 @@
 				    <mesh filename="package://sef_roboter_support/meshes/sr25/visual/sr25_axis_tool.stl" />
 			      </geometry>
-			      <material name="black" />
+            <material name="grey" />
 		      </visual>
 		      <collision>

Commit message: fixing position limit for joint 1

File: sef_roboter_support/urdf/sr25_macro.xacro (robot description, xacro)
@@ -171,5 +171,5 @@
 			<origin xyz="0 0 0.075738" rpy="1.5708 0 -1.5745"/>
 			<axis xyz="0 -1 0" />
-			<limit lower="-2.8" upper="2.8" effort="10000" velocity="1" />
+                        <limit lower="-1" upper="1" velocity="1" />
  			<dynamics damping="0.7" friction="100"/>
 	      </joint>
@@ -179,5 +179,5 @@
 			<origin xyz="0 0.24264 -0.29599" rpy="1.5687 0 0"/>
 			<axis xyz="-1 0 0" />
-                        <limit lower="-0.5" upper="1.5" effort="10000" velocity="1" />
+                        <limit lower="-0.5" upper="1.5" velocity="1" />
 			<dynamics damping="0.7" friction="100"/>
 	      </joint>
@@ -187,5 +187,5 @@
 			<origin xyz="0 0 -0.79724" rpy="0.005529 0 0"/>
 			<axis xyz="-1 0 0" />
-                        <limit lower="-1.5" upper="0.5" effort="10000" velocity="1" />
+                        <limit lower="-1.5" upper="0.5" velocity="1" />
 		        <dynamics damping="0.7" friction="100"/>
 	      </joint>
@@ -195,5 +195,5 @@
 			<origin xyz="0 -0.15811 0" rpy="0 0.0014787 0"/>
 			<axis xyz="0 1 0" />
-                        <limit lower="-3" upper="3" effort="10000" velocity="1" />
+                        <limit lower="-3" upper="3" velocity="1" />
 			<dynamics damping="0.7" friction="100"/>
               </joint>
@@ -203,5 +203,5 @@
 			<origin xyz="0 -0.58433 0" rpy="0 0 -0.033693"/>
 			<axis xyz="0 0 1" />
-                        <limit lower="-1.6" upper="1.6" effort="10000" velocity="1" />
+                        <limit lower="-1.6" upper="1.6" velocity="1" />
 			<dynamics damping="0.7" friction="100"/>
               </joint>
@@ -211,5 +211,5 @@
 			<origin xyz="0 -0.164051291252016 -0.00548103448275694" rpy="-1.5707963267949 0 3.14159265358979"/>
 			<axis xyz="0 0 -1 " />
-			<limit lower="-2.5" upper="2.5" effort="100" velocity="1" />
+                        <limit lower="-2.5" upper="2.5" velocity="1" />
 			<dynamics damping="0.7" friction="100"/>
               </joint>

Commit message: tuned urdf params

File: sef_roboter_support/urdf/sr25_macro.xacro (robot description, xacro)
@@ -171,6 +171,6 @@
 			<origin xyz="0 0 0.075738" rpy="1.5708 0 -1.5745"/>
 			<axis xyz="0 -1 0" />
-                        <limit lower="-1" upper="1" velocity="1" />
- 			<dynamics damping="0.7" friction="100"/>
+                        <limit lower="-1" upper="1" effort="5000" velocity="1" />
+                        <dynamics damping="2"/>
 	      </joint>
 	      <joint name="${prefix}joint_2" type="revolute">
@@ -179,6 +179,6 @@
 			<origin xyz="0 0.24264 -0.29599" rpy="1.5687 0 0"/>
 			<axis xyz="-1 0 0" />
-                        <limit lower="-0.5" upper="1.5" velocity="1" />
-			<dynamics damping="0.7" friction="100"/>
+                        <limit lower="-0.5" upper="1.5" effort="5000" velocity="1" />
+                        <dynamics damping="2"/>
 	      </joint>
 	      <joint name="${prefix}joint_3" type="revolute">
@@ -187,6 +187,6 @@
 			<origin xyz="0 0 -0.79724" rpy="0.005529 0 0"/>
 			<axis xyz="-1 0 0" />
-                        <limit lower="-1.5" upper="0.5" velocity="1" />
-		        <dynamics damping="0.7" friction="100"/>
+                        <limit lower="-1.5" upper="0.5" effort="5000" velocity="1" />
+                        <dynamics damping="2"/>
 	      </joint>
 	      <joint name="${prefix}joint_4" type="revolute">
@@ -195,6 +195,6 @@
 			<origin xyz="0 -0.15811 0" rpy="0 0.0014787 0"/>
 			<axis xyz="0 1 0" />
-                        <limit lower="-3" upper="3" velocity="1" />
-			<dynamics damping="0.7" friction="100"/>
+                        <limit lower="-3" upper="3" effort="5000" velocity="1" />
+                        <dynamics damping="2"/>
               </joint>
 	      <joint name="${prefix}joint_5" type="revolute">
@@ -203,6 +203,6 @@
 			<origin xyz="0 -0.58433 0" rpy="0 0 -0.033693"/>
 			<axis xyz="0 0 1" />
-                        <limit lower="-1.6" upper="1.6" velocity="1" />
-			<dynamics damping="0.7" friction="100"/>
+                        <limit lower="-1.6" upper="1.6" effort="5000" velocity="1" />
+                        <dynamics damping="2"/>
               </joint>
 	      <joint name="${prefix}joint_6" type="revolute">
@@ -211,6 +211,6 @@
 			<origin xyz="0 -0.164051291252016 -0.00548103448275694" rpy="-1.5707963267949 0 3.14159265358979"/>
 			<axis xyz="0 0 -1 " />
-                        <limit lower="-2.5" upper="2.5" velocity="1" />
-			<dynamics damping="0.7" friction="100"/>
+                        <limit lower="-2.5" upper="2.5" effort="5000" velocity="1" />
+                        <dynamics damping="2" />
               </joint>
 	      <!-- end of joint list -->
